File: spider.sch (KiCad schematic (older format))
At the start: 19 parts, among them IC1 ATMEGA88-A, J1 CONN_02X04, P2 USB_OTG, P3 CONN_01X01, U1 ESP8266-ESP-03, U2 nRF24L01+, U3 LD1117S33TR, U4 HS0038

Commit message: Add more expansion pins, route 5V to transmitter, add small fixes.
Parts:
- removed J1: CONN_02X04, Pin_Headers:Pin_Header_Straight_2x04_Pitch2.54mm, symbol CONN_02X04
- added J1: CONN_02X05, Pin_Headers:Pin_Header_Straight_2x05_Pitch2.54mm, symbol CONN_02X05
- P2: footprint spider:USB_Micro-B -> spider:USB_Micro-B handsoldering
- RF2: value RF_Transmitter_433_MHz -> 433 MHz
Connections:
- net 5V: now also J1.8 (P8)
- net ADCin: now also J1.7 (P7)
- net GND: now also J1.6 (P6)
- net MISO: now also J1.1 (P1)
- net MOSI: now also J1.4 (P4)
- net SCK: now also J1.3 (P3)
- net VCC: now also J1.2 (P2)
- net ~RST: now also J1.5 (P5)
- net espTX: now reaches IC1.30 ((PCINT16/RXD)PD0), U1.3 (TX)
- net espTX: now also J1.10 (P10)
- net espRX: now reaches IC1.31 ((PCINT17/TXD)PD1), U1.4 (RX)
- net espRX: now also J1.9 (P9)
Changed lines of the file:
@@
 P 4700 5225
 F 0 "RF2" H 4725 5750 60  0000 C CNN
-F 1 "RF_Transmitter_433_MHz" H 4825 4925 60  0001 C CNN
+F 1 "433 MHz" H 4825 4925 60  0001 C CNN
 F 2 "spider:RF_Transmitter_433_MHz" H 4700 5225 60  0001 C CNN
 F 3 "" H 4700 5225 60  0000 C CNN
@@
 F 0 "P2" H 6050 750 50  0000 C CNN
 F 1 "USB_OTG" H 5725 1075 50  0000 C CNN
-F 2 "spider:USB_Micro-B" V 5375 800 50  0001 C CNN
+F 2 "spider:USB_Micro-B handsoldering" V 5375 800 50  0001 C CNN
 F 3 "" V 5675 775 50  0000 C CNN
 	1    5725 875
@@
 Text Label 3925 1450 0    60   ~ 0
 5V
-$Comp
-L CONN_02X04 J1
-U 1 1 58DD8F64
-P 3675 1300
-F 0 "J1" H 3675 1550 50  0000 C CNN
-F 1 "CONN_02X04" H 3675 1050 50  0000 C CNN
-F 2 "Pin_Headers:Pin_Header_Straight_2x04_Pitch2.54mm" H 3675 100 50  0001 C CNN
-F 3 "" H 3675 100 50  0001 C CNN
-	1    3675 1300
-	1    0    0    -1
-$EndComp
 NoConn ~ 1250 3450
 Text Label 3150 3350 0    60   ~ 0
@@
 Wire Wire Line
 	3350 3250 3150 3250
+Text Label 3725 3700 1    60   ~ 0
+espTX
+Text Label 3725 3800 3    60   ~ 0
+espRX
+Connection ~ 3725 3800
+Connection ~ 3725 3700
+$Comp
+L CONN_02X05 J1
+U 1 1 58E122B1
+P 3675 1350
+F 0 "J1" H 3675 1650 50  0000 C CNN
+F 1 "CONN_02X05" H 3675 1050 50  0000 C CNN
+F 2 "Pin_Headers:Pin_Header_Straight_2x05_Pitch2.54mm" H 3675 150 50  0001 C CNN
+F 3 "" H 3675 150 50  0001 C CNN
+	1    3675 1350
+	1    0    0    -1
+$EndComp
+Text Label 3925 1550 0    60   ~ 0
+espTX
+Text Label 3425 1550 2    60   ~ 0
+espRX
 $EndSCHEMATC
